Commit message: Updating puma_resources

File: puma_resources/urdf/puma.urdf (robot description, URDF)
Before this commit: robot puma, 9 links, 8 joints
Links:
- link map: geometry visual mesh filename=package://lab2/meshes/base.stl scale=1 1 1
- link {s}: geometry 
Joints:
- removed joint 6_to_b
- added joint jointb: type fixed, parent {6}, child {b}, origin xyz=0 0 0 rpy=1.57 0 -1.57, axis 0 0 1
- joint joint2: limit lower=-1.57 upper=1.57 effort=100.0 velocity=2.0 -> lower=-3.14 upper=3.14 effort=100.0 velocity=2.0; origin xyz=0 0 0 rpy=0 0 0 -> xyz=0.14 0 0 rpy=0 1.57 0
- joint joint3: limit lower=-1.57 upper=1.57 effort=100.0 velocity=2.0 -> lower=-3.14 upper=3.14 effort=100.0 velocity=2.0; origin xyz=0 0 0 rpy=0 0 0 -> xyz=0 0.45 0 rpy=0 0 0
- joint joint4: limit lower=-1.57 upper=1.57 effort=100.0 velocity=2.0 -> lower=-3.14 upper=3.14 effort=100.0 velocity=2.0; origin xyz=0 0 0 rpy=0 0 0 -> xyz=0 0.49 0 rpy=-1.57 0 0
- joint joint5: limit lower=-1.57 upper=1.57 effort=100.0 velocity=2.0 -> lower=-3.14 upper=3.14 effort=100.0 velocity=2.0; origin xyz=0 0 0 rpy=0 0 0 -> xyz=0 0 0 rpy=1.57 0 0
- joint joint6: limit lower=-1.57 upper=1.57 effort=100.0 velocity=2.0 -> lower=-3.14 upper=3.14 effort=100.0 velocity=2.0; origin xyz=0 0 0 rpy=0 0 0 -> xyz=0 0 0 rpy=-1.57 0 0
- joint map_to_s: origin xyz=0 0 0 rpy=0 0 0 -> xyz=0 0 0.623 rpy=0 0 0

Commit message: Some puma_resources fixes.

File: puma_resources/urdf/puma.urdf (robot description, URDF)
Before this commit: robot puma, 9 links, 8 joints
Links:
- link map: geometry visual mesh filename=package://puma_description/meshes/base.stl scale=1 1 1
- link {1}: geometry visual mesh filename=package://puma_description/meshes/link1.stl scale=1 1 1
- link {2}: geometry visual mesh filename=package://puma_description/meshes/link2.stl scale=1 1 1
- link {3}: geometry visual mesh filename=package://puma_description/meshes/link3.stl scale=1 1 1
- link {4}: geometry visual mesh filename=package://puma_description/meshes/link4.stl scale=1 1 1
- link {5}: geometry visual mesh filename=package://puma_description/meshes/link5.stl scale=1 1 1
